File: PCB Design/SRMAD_PCB_KiCAD_Files/IoT_Deployement_Board.sch (KiCad schematic (older format))
At the start: 64 parts, among them J1 PWR, J10 DHT22, J11 DS18B20, J2 Switch_Conn, J3 Soil_Moisture, J4 LED_CONN, J5 Pump_Conn, J6 BH1750, J7 HTUI2D, J8 Prog_Header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

Commit message: Added Enclosure V2 build-in-progress
Parts:
- R23: value 0805 -> 470e
Changed lines of the file:
@@
 encoding utf-8
 Sheet 1 1
-Title "IoT Plant Monitoring and Watering System"
+Title "ESP32_based_IoT_Deployement_Board"
 Date ""
 Rev "v0.1"
@@
 U 1 1 5FE059EE
 P 6850 5700
-F 0 "R23" H 6700 5800 45  0000 C CNN
-F 1 "0805" H 6850 5800 45  0000 C CNN
+F 0 "R23" H 6850 5800 45  0000 C CNN
+F 1 "470e" H 6850 5600 45  0000 C CNN
 F 2 "0805" H 6850 5850 20  0001 C CNN
 F 3 "" H 6850 5700 60  0001 C CNN
